File: pcb/k6_carrier_rev2.kicad_pcb (KiCad board)
At the start: 2 copper layers, 100 x 80 mm, 31 parts, among them J1 12V_DC, J2 48V_DC, SW1 RING, SW2 CANCEL, SW3 RESET, SW4 MODE, T1 600R_XFMR, U1 PC817, U2 L293D

Commit message: fix: correct transformer, DAC, and R1 footprints
- Transformer T1: 2x2 pin header matching EI-14 audio transformer
- DAC: added 2-pin screw terminal (J_SPK) for speaker output
- R1: same pad size as R2/R3 for consistency (was using larger 1W footprint)

Co-Authored-By: Devin AI <158243242+devin-ai-integration[bot]@users.noreply.github.com>
Parts:
- added J_SPK: Speaker, TerminalBlock_bornier-2_P5.08mm, F.Cu at (110.0, 90.0)
- R1: value 470R -> 470R_1W; footprint R_Axial_DIN0309_L9.0mm_D3.2mm_P12.70mm_Horizontal -> R_Axial_DIN0207_L6.3mm_D2.5mm_P7.62mm_Horizontal
- T1: footprint PinHeader_1x04_P2.54mm_Vertical -> PinHeader_2x02_P2.54mm_Vertical
- moved T1 4.00 mm to (120.0, 96.0)
Other:
- board text added: "Pri Sec"
- board text added: "SPK+/-"
